File: avr-programmer.kicad_pcb (KiCad board)
At the start: 2 copper layers, 57.4 x 66.3 mm, 6 parts, among them J1 AVR-ISP-6, J2 Conn_01x15_Male, J3 Conn_01x15_Male, Q1 2N7000, U1 ATmega328P-PU

Commit message: udating everything I guess!
Parts:
- added C2: 10uf, Capacitor_THT:CP_Radial_D5.0mm_P2.00mm, F.Cu at (131.6, 123.2)
- added J4: USB_B_Mini, Connector_USB:USB_Mini-B_Lumberg_2486_01_Horizontal, F.Cu at (146.8, 71.4)
- added J5: Conn_01x02_Male, Connector_PinHeader_2.54mm:PinHeader_1x02_P2.54mm_Vertical, F.Cu at (158.0, 124.0)
- added U2: LD1117S33TR_SOT223, Package_TO_SOT_THT:TO-220-3_Horizontal_TabDown, F.Cu at (123.7, 128.5)
- moved Q1 17.2 mm to (131.3, 127.8)
- moved J1 13.5 mm to (142.7, 127.5)
Routing:
- net +5V: track 76.7 -> 128.8 mm
- net +3V3: track 0.00 -> 47.6 mm
- net GNDA: track 56.3 -> 74.6 mm
- net Net-(J1-Pad5): track 97.2 -> 103.5 mm
- net Net-(J1-Pad4): track 42.4 -> 45.5 mm
- net Net-(J1-Pad3): track 51.0 -> 53.5 mm
- net Net-(J1-Pad1): track 49.2 -> 51.2 mm, vias 0 -> 1
Other:
- board text added: "3.3V"
