File: avr-programmer.sch (KiCad schematic (older format))
At the start: 6 parts, among them J1 AVR-ISP-6, J2 Conn_01x15_Male, J3 Conn_01x15_Male, Q1 2N7000, U1 ATmega328P-PU

Commit message: udating everything I guess!
Parts:
- added C2: 10uf, Capacitor_THT:CP_Radial_D5.0mm_P2.00mm, symbol Device:CP1
- added J4: USB_B_Mini, Connector_USB:USB_Mini-B_Lumberg_2486_01_Horizontal, symbol Connector:USB_B_Mini
- added J5: Conn_01x02_Male, Connector_PinHeader_2.54mm:PinHeader_1x02_P2.54mm_Vertical, symbol Connector:Conn_01x02_Male
- added U2: LD1117S33TR_SOT223, Package_TO_SOT_THT:TO-220-3_Horizontal_TabDown, symbol Regulator_Linear:LD1117S33TR_SOT223
Connections:
- net +5V: now also J4.1 (VBUS), U2.3 (VI)
- net GND: now also C2.2, J4.5 (GND), J5.1 (Pin_1), U2.1 (GND)
- new net +3V3: C2.1, J5.2 (Pin_2), U2.2 (VO)
Changed lines of the file:
@@
 	5350 5000 5700 5000
 $Comp
-L power:GND #PWR?
+L power:GND #PWR0113
 U 1 1 5E76F274
 P 1150 5350
-F 0 "#PWR?" H 1150 5100 50  0001 C CNN
+F 0 "#PWR0113" H 1150 5100 50  0001 C CNN
 F 1 "GND" H 1155 5177 50  0000 C CNN
 F 2 "" H 1150 5350 50  0001 C CNN
@@
 Wire Wire Line
 	1600 5350 1150 5350
+$Comp
+L Regulator_Linear:LD1117S33TR_SOT223 U2
+U 1 1 5E71D845
+P 8650 3250
+F 0 "U2" H 8650 3492 50  0000 C CNN
+F 1 "LD1117S33TR_SOT223" H 8650 3401 50  0000 C CNN
+F 2 "Package_TO_SOT_THT:TO-220-3_Horizontal_TabDown" H 8650 3450 50  0001 C CNN
+F 3 "http://www.st.com/st-web-ui/static/active/en/resource/technical/document/datasheet/CD00000544.pdf" H 8750 3000 50  0001 C CNN
+	1    8650 3250
+	1    0    0    -1
+$EndComp
+$Comp
+L power:+5V #PWR0114
+U 1 1 5E71F0E2
+P 8350 2900
+F 0 "#PWR0114" H 8350 2750 50  0001 C CNN
+F 1 "+5V" H 8365 3073 50  0000 C CNN
+F 2 "" H 8350 2900 50  0001 C CNN
+F 3 "" H 8350 2900 50  0001 C CNN
+	1    8350 2900
+	1    0    0    -1
+$EndComp
+Wire Wire Line
+	8350 3250 8350 2900
+$Comp
+L power:GND #PWR0115
+U 1 1 5E723BEC
+P 8650 3750
+F 0 "#PWR0115" H 8650 3500 50  0001 C CNN
+F 1 "GND" H 8655 3577 50  0000 C CNN
+F 2 "" H 8650 3750 50  0001 C CNN
+F 3 "" H 8650 3750 50  0001 C CNN
+	1    8650 3750
+	1    0    0    -1
+$EndComp
+Wire Wire Line
+	8650 3550 8650 3750
+$Comp
+L power:+3.3V #PWR0116
+U 1 1 5E72846D
+P 8950 2900
+F 0 "#PWR0116" H 8950 2750 50  0001 C CNN
+F 1 "+3.3V" H 8965 3073 50  0000 C CNN
+F 2 "" H 8950 2900 50  0001 C CNN
+F 3 "" H 8950 2900 50  0001 C CNN
+	1    8950 2900
+	1    0    0    -1
+$EndComp
+Wire Wire Line
+	8950 3250 8950 2900
+$Comp
+L Device:CP1 C2
+U 1 1 5E72D09E
+P 7250 5300
+F 0 "C2" H 7365 5346 50  0000 L CNN
+F 1 "10uf" H 7365 5255 50  0000 L CNN
+F 2 "Capacitor_THT:CP_Radial_D5.0mm_P2.00mm" H 7250 5300 50  0001 C CNN
+F 3 "~" H 7250 5300 50  0001 C CNN
+	1    7250 5300
+	1    0    0    -1
+$EndComp
+$Comp
+L power:GND #PWR0117
+U 1 1 5E72DA22
+P 7250 5600
+F 0 "#PWR0117" H 7250 5350 50  0001 C CNN
+F 1 "GND" H 7255 5427 50  0000 C CNN
+F 2 "" H 7250 5600 50  0001 C CNN
+F 3 "" H 7250 5600 50  0001 C CNN
+	1    7250 5600
+	1    0    0    -1
+$EndComp
+$Comp
+L power:+3.3V #PWR0118
+U 1 1 5E72DF70
+P 7250 4950
+F 0 "#PWR0118" H 7250 4800 50  0001 C CNN
+F 1 "+3.3V" H 7265 5123 50  0000 C CNN
+F 2 "" H 7250 4950 50  0001 C CNN
+F 3 "" H 7250 4950 50  0001 C CNN
+	1    7250 4950
+	1    0    0    -1
+$EndComp
+Wire Wire Line
+	7250 5150 7250 4950
+Wire Wire Line
+	7250 5450 7250 5600
+$Comp
+L Connector:USB_B_Mini J4
+U 1 1 5E7370FE
+P 8500 5150
+F 0 "J4" H 8557 5617 50  0000 C CNN
+F 1 "USB_B_Mini" H 8557 5526 50  0000 C CNN
+F 2 "Connector_USB:USB_Mini-B_Lumberg_2486_01_Horizontal" H 8650 5100 50  0001 C CNN
+F 3 "~" H 8650 5100 50  0001 C CNN
+	1    8500 5150
+	1    0    0    -1
+$EndComp
+$Comp
+L power:GND #PWR0119
+U 1 1 5E737D22
+P 8500 5800
+F 0 "#PWR0119" H 8500 5550 50  0001 C CNN
+F 1 "GND" H 8505 5627 50  0000 C CNN
+F 2 "" H 8500 5800 50  0001 C CNN
+F 3 "" H 8500 5800 50  0001 C CNN
+	1    8500 5800
+	1    0    0    -1
+$EndComp
+Wire Wire Line
+	8500 5550 8500 5800
+$Comp
+L power:+5V #PWR0120
+U 1 1 5E73C8C1
+P 8950 4800
+F 0 "#PWR0120" H 8950 4650 50  0001 C CNN
+F 1 "+5V" H 8965 4973 50  0000 C CNN
+F 2 "" H 8950 4800 50  0001 C CNN
+F 3 "" H 8950 4800 50  0001 C CNN
+	1    8950 4800
+	1    0    0    -1
+$EndComp
+Wire Wire Line
+	8800 4950 8950 4950
+Wire Wire Line
+	8950 4950 8950 4800
+$Comp
+L Connector:Conn_01x02_Male J5
+U 1 1 5E751A90
+P 9700 4550
+F 0 "J5" H 9808 4731 50  0000 C CNN
+F 1 "Conn_01x02_Male" H 9808 4640 50  0000 C CNN
+F 2 "Connector_PinHeader_2.54mm:PinHeader_1x02_P2.54mm_Vertical" H 9700 4550 50  0001 C CNN
+F 3 "~" H 9700 4550 50  0001 C CNN
+	1    9700 4550
+	1    0    0    -1
+$EndComp
+$Comp
+L power:+3.3V #PWR0121
+U 1 1 5E75262D
+P 9900 4800
+F 0 "#PWR0121" H 9900 4650 50  0001 C CNN
+F 1 "+3.3V" H 9915 4973 50  0000 C CNN
+F 2 "" H 9900 4800 50  0001 C CNN
+F 3 "" H 9900 4800 50  0001 C CNN
+	1    9900 4800
+	-1   0    0    1
+$EndComp
+$Comp
+L power:GND #PWR0122
+U 1 1 5E75784D
+P 9900 4300
+F 0 "#PWR0122" H 9900 4050 50  0001 C CNN
+F 1 "GND" H 9905 4127 50  0000 C CNN
+F 2 "" H 9900 4300 50  0001 C CNN
+F 3 "" H 9900 4300 50  0001 C CNN
+	1    9900 4300
+	-1   0    0    1
+$EndComp
+Wire Wire Line
+	9900 4550 9900 4300
+Wire Wire Line
+	9900 4650 9900 4800
 $EndSCHEMATC
